File: rocketShip/rocketShip.kicad_pcb (KiCad board)
At the start: 2 copper layers, 59.5 x 105.8 mm, 18 parts, among them Q1 NPN, Q2 NPN, Q3 NPN, SW1 SW_Push

Commit message: added some back art
Parts:
- added G***: LOGO, LOGO, B.Cu at (100.0, 125.5)
